Commit message: refactor(my_robot_description): keep nero baseline only

File: nero/urdf/nero_description.urdf (robot description, URDF)
Before this commit: robot nero, 9 links, 8 joints
Links:
- link base_link: geometry collision mesh filename=package://agx_arm_description/nero/meshes/base_link.stl; visual mesh filename=package://agx_arm_description/nero/meshes/dae/base_link.dae
- link link1: geometry collision mesh filename=package://agx_arm_description/nero/meshes/link1.stl; visual mesh filename=package://agx_arm_description/nero/meshes/dae/link1.dae
- link link2: geometry collision mesh filename=package://agx_arm_description/nero/meshes/link2.stl; visual mesh filename=package://agx_arm_description/nero/meshes/dae/link2.dae
- link link3: geometry collision mesh filename=package://agx_arm_description/nero/meshes/link3.stl; visual mesh filename=package://agx_arm_description/nero/meshes/dae/link3.dae
- link link4: geometry collision mesh filename=package://agx_arm_description/nero/meshes/link4.stl; visual mesh filename=package://agx_arm_description/nero/meshes/dae/link4.dae
- link link5: geometry collision mesh filename=package://agx_arm_description/nero/meshes/link5.stl; visual mesh filename=package://agx_arm_description/nero/meshes/dae/link5.dae
- link link6: geometry collision mesh filename=package://agx_arm_description/nero/meshes/link6.stl; visual mesh filename=package://agx_arm_description/nero/meshes/dae/link6.dae
- link link7: geometry collision mesh filename=package://agx_arm_description/nero/meshes/link7.stl; visual mesh filename=package://agx_arm_description/nero/meshes/dae/link7.dae

File: nero/urdf/nero_with_gripper_description.xacro (robot description, xacro)
@@ -3,5 +3,5 @@
      For more information, please see http://wiki.ros.org/sw_urdf_exporter -->
 <robot xmlns:xacro="http://www.ros.org/wiki/xacro" name="nero">
-<xacro:include filename="$(find agx_arm_description)/agx_arm_urdf/nero/urdf/nero_with_gripper_flange_description.xacro"/>
+<xacro:include filename="$(find agx_arm_description)/nero/urdf/nero_with_gripper_flange_description.xacro"/>
     <link name="gripper_base">
         <inertial>
@@ -13,5 +13,5 @@
             <origin xyz="0 0 0" rpy="0 0 0"/>
             <geometry>
-                <mesh filename="package://agx_arm_description/agx_arm_urdf/nero/meshes/dae/gripper_base.dae"/>
+                <mesh filename="package://agx_arm_description/nero/meshes/dae/gripper_base.dae"/>
             </geometry>
         </visual>
@@ -19,5 +19,5 @@
             <origin xyz="0 0 0" rpy="0 0 0"/>
             <geometry>
-                <mesh filename="package://agx_arm_description/agx_arm_urdf/nero/meshes/gripper_base.stl"/>
+                <mesh filename="package://agx_arm_description/nero/meshes/gripper_base.stl"/>
             </geometry>
         </collision>
@@ -37,5 +37,5 @@
             <origin xyz="0 0 0" rpy="0 0 0"/>
             <geometry>
-                <mesh filename="package://agx_arm_description/agx_arm_urdf/nero/meshes/dae/gripper_link1.dae"/>
+                <mesh filename="package://agx_arm_description/nero/meshes/dae/gripper_link1.dae"/>
             </geometry>
         </visual>
@@ -43,5 +43,5 @@
             <origin xyz="0 0 0" rpy="0 0 0"/>
             <geometry>
-                <mesh filename="package://agx_arm_description/agx_arm_urdf/nero/meshes/gripper_link1.stl"/>
+                <mesh filename="package://agx_arm_description/nero/meshes/gripper_link1.stl"/>
             </geometry>
         </collision>
@@ -63,5 +63,5 @@
             <origin xyz="0 0 0" rpy="0 0 0"/>
             <geometry>
-                <mesh filename="package://agx_arm_description/agx_arm_urdf/nero/meshes/dae/gripper_link2.dae"/>
+                <mesh filename="package://agx_arm_description/nero/meshes/dae/gripper_link2.dae"/>
             </geometry>
         </visual>
@@ -69,5 +69,5 @@
             <origin xyz="0 0 0" rpy="0 0 0"/>
             <geometry>
-                <mesh filename="package://agx_arm_description/agx_arm_urdf/nero/meshes/gripper_link2.stl"/>
+                <mesh filename="package://agx_arm_description/nero/meshes/gripper_link2.stl"/>
             </geometry>
         </collision>

File: nero/urdf/nero_with_gripper_flange_description.xacro (robot description, xacro)
@@ -3,5 +3,5 @@
      For more information, please see http://wiki.ros.org/sw_urdf_exporter -->
 <robot xmlns:xacro="http://www.ros.org/wiki/xacro" name="nero">
-<xacro:include filename="$(find agx_arm_description)/agx_arm_urdf/nero/urdf/nero_description.urdf"/>
+<xacro:include filename="$(find agx_arm_description)/nero/urdf/nero_description.urdf"/>
     <link name="gripper_flange">
         <inertial>
@@ -13,5 +13,5 @@
             <origin xyz="0 0 0" rpy="0 0 0"/>
             <geometry>
-                <mesh filename="package://agx_arm_description/agx_arm_urdf/nero/meshes/dae/gripper_flange.dae"/>
+                <mesh filename="package://agx_arm_description/nero/meshes/dae/gripper_flange.dae"/>
             </geometry>
         </visual>
@@ -19,5 +19,5 @@
             <origin xyz="0 0 0" rpy="0 0 0"/>
             <geometry>
-                <mesh filename="package://agx_arm_description/agx_arm_urdf/nero/meshes/gripper_flange.stl"/>
+                <mesh filename="package://agx_arm_description/nero/meshes/gripper_flange.stl"/>
             </geometry>
         </collision>

File: nero/urdf/nero_with_left_revo2_description.xacro (robot description, xacro)
@@ -4,6 +4,6 @@
      For more information, please see http://wiki.ros.org/sw_urdf_exporter -->
 <robot xmlns:xacro="http://www.ros.org/wiki/xacro" name="nero">
-<xacro:include filename="$(find agx_arm_description)/agx_arm_urdf/revo2/urdf/revo2_left_hand.urdf"/>
-<xacro:include filename="$(find agx_arm_description)/agx_arm_urdf/nero/urdf/nero_with_revo2_flange_description.xacro"/>
+<xacro:include filename="$(find agx_arm_description)/revo2/urdf/revo2_left_hand.urdf"/>
+<xacro:include filename="$(find agx_arm_description)/nero/urdf/nero_with_revo2_flange_description.xacro"/>
     <joint name="hand_base_joint" type="fixed">
         <origin xyz="0.0 0.0 0.012" rpy="0 0 3.1415926"/>

File: nero/urdf/nero_with_revo2_flange_description.xacro (robot description, xacro)
@@ -3,5 +3,5 @@
      For more information, please see http://wiki.ros.org/sw_urdf_exporter -->
 <robot xmlns:xacro="http://www.ros.org/wiki/xacro" name="nero">
-<xacro:include filename="$(find agx_arm_description)/agx_arm_urdf/nero/urdf/nero_description.urdf"/>
+<xacro:include filename="$(find agx_arm_description)/nero/urdf/nero_with_gripper_flange_description.xacro"/>
     <link name="revo2_flange">
         <inertial>
@@ -13,5 +13,5 @@
             <origin xyz="0 0 0" rpy="0 0 0"/>
             <geometry>
-                <mesh filename="package://agx_arm_description/agx_arm_urdf/nero/meshes/dae/revo2_flange.dae"/>
+                <mesh filename="package://agx_arm_description/nero/meshes/dae/revo2_flange.dae"/>
             </geometry>
         </visual>
@@ -19,5 +19,5 @@
             <origin xyz="0 0 0" rpy="0 0 0"/>
             <geometry>
-                <mesh filename="package://agx_arm_description/agx_arm_urdf/nero/meshes/revo2_flange.stl"/>
+                <mesh filename="package://agx_arm_description/nero/meshes/revo2_flange.stl"/>
             </geometry>
         </collision>

File: nero/urdf/nero_with_right_revo2_description.xacro (robot description, xacro)
@@ -4,6 +4,6 @@
      For more information, please see http://wiki.ros.org/sw_urdf_exporter -->
 <robot xmlns:xacro="http://www.ros.org/wiki/xacro" name="nero">
-<xacro:include filename="$(find agx_arm_description)/agx_arm_urdf/revo2/urdf/revo2_right_hand.urdf"/>
-<xacro:include filename="$(find agx_arm_description)/agx_arm_urdf/nero/urdf/nero_with_revo2_flange_description.xacro"/>
+<xacro:include filename="$(find agx_arm_description)/revo2/urdf/revo2_right_hand.urdf"/>
+<xacro:include filename="$(find agx_arm_description)/nero/urdf/nero_with_revo2_flange_description.xacro"/>
     <joint name="hand_base_joint" type="fixed">
         <origin xyz="0.0 0.0 0.012" rpy="0 0 3.1415926"/>
