Commit message: fix(my_robot_description): widen nero joint limits for hardware validation

File: urdf/robots/nero/nero_description.urdf (robot description, URDF)
Before this commit: robot nero, 9 links, 8 joints
Joints:
- joint joint2: limit lower=-1.74 upper=1.74 effort=100 velocity=5 -> lower=-1.80 upper=1.80 effort=100 velocity=5
- joint joint4: limit lower=-1.01 upper=2.14 effort=100 velocity=5 -> lower=-1.01 upper=2.20 effort=100 velocity=5

File: urdf/variants/nero_blade_polishing/nero_blade_polishing.urdf (robot description, URDF)
Before this commit: robot nero_blade_polishing, 25 links, 24 joints
Joints:
- joint joint2: limit lower=-1.74 upper=1.74 effort=100 velocity=5 -> lower=-1.80 upper=1.80 effort=100 velocity=5
- joint joint4: limit lower=-1.01 upper=2.14 effort=100 velocity=5 -> lower=-1.01 upper=2.20 effort=100 velocity=5

File: urdf/variants/nero_blade_polishing/nero_blade_polishing_tesseract.urdf (robot description, URDF)
Before this commit: robot nero_blade_polishing, 25 links, 24 joints
Joints:
- joint joint2: limit lower=-1.74 upper=1.74 effort=100 velocity=5 -> lower=-1.80 upper=1.80 effort=100 velocity=5
- joint joint4: limit lower=-1.01 upper=2.14 effort=100 velocity=5 -> lower=-1.01 upper=2.20 effort=100 velocity=5
