Commit message: fix(my_robot_description): align blade polishing TCP model

File: urdf/end_effectors/end_effector_with_tcp.xacro (robot description, xacro)
@@ -17,5 +17,5 @@
         </link>
         <joint name="gripper_flange_to_end_effector_joint" type="fixed">
-            <origin xyz="0 0 0.01" rpy="0 3.1415926535897 -1.5707963268"/>
+            <origin xyz="0 0 0.01" rpy="0 3.1415926535897 1.5707963268"/>
             <parent link="${parent}"/>
             <child link="end_effector_link"/>
@@ -23,5 +23,5 @@
         <link name="polishing_tcp"/>
         <joint name="end_effector_to_polishing_tcp_joint" type="fixed">
-            <origin xyz="0 -0.05085 -0.20074" rpy="0 0 3.14159265358979"/>
+            <origin xyz="0 -0.05085 -0.20074" rpy="3.14159265358979 0 3.14159265358979"/>
             <parent link="end_effector_link"/>
             <child link="polishing_tcp"/>

File: urdf/variants/nero_blade_polishing/nero_blade_polishing.urdf (robot description, URDF)
Before this commit: robot nero_blade_polishing, 25 links, 24 joints
Joints:
- joint end_effector_to_polishing_tcp_joint: origin xyz=0 -0.05085 -0.20074 rpy=0 0 3.14159265358979 -> xyz=0 -0.05085 -0.20074 rpy=3.14159265358979 0 3.14159265358979
- joint gripper_flange_to_end_effector_joint: origin xyz=0 0 0.01 rpy=0 3.1415926535897 -1.5707963268 -> xyz=0 0 0.01 rpy=0 3.1415926535897 1.5707963268

File: urdf/variants/nero_blade_polishing/nero_blade_polishing_tesseract.urdf (robot description, URDF)
Before this commit: robot nero_blade_polishing, 25 links, 24 joints
Joints:
- joint end_effector_to_polishing_tcp_joint: origin xyz=0 -0.05085 -0.20074 rpy=0 0 3.14159265358979 -> xyz=0 -0.05085 -0.20074 rpy=3.14159265358979 0 3.14159265358979
- joint gripper_flange_to_end_effector_joint: origin xyz=0 0 0.01 rpy=0 3.1415926535897 -1.5707963268 -> xyz=0 0 0.01 rpy=0 3.1415926535897 1.5707963268
