Commit message: fix(my_robot_description): align blade polishing frames

File: urdf/end_effectors/end_effector_with_tcp.xacro (robot description, xacro)
@@ -23,5 +23,5 @@
         <link name="polishing_tcp"/>
         <joint name="end_effector_to_polishing_tcp_joint" type="fixed">
-            <origin xyz="0 -0.05085 -0.20074" rpy="3.14159265358979 0 3.14159265358979"/>
+            <origin xyz="0 -0.05085 -0.19574" rpy="3.14159265358979 0 3.14159265358979"/>
             <parent link="end_effector_link"/>
             <child link="polishing_tcp"/>

File: urdf/variants/nero_blade_polishing/nero_blade_polishing.urdf (robot description, URDF)
Before this commit: robot nero_blade_polishing, 25 links, 24 joints
Joints:
- joint end_effector_to_polishing_tcp_joint: origin xyz=0 -0.05085 -0.20074 rpy=3.14159265358979 0 3.14159265358979 -> xyz=0 -0.05085 -0.19574 rpy=3.14159265358979 0 3.14159265358979

File: urdf/variants/nero_blade_polishing/nero_blade_polishing_tesseract.urdf (robot description, URDF)
Before this commit: robot nero_blade_polishing, 25 links, 24 joints
Joints:
- joint end_effector_to_polishing_tcp_joint: origin xyz=0 -0.05085 -0.20074 rpy=3.14159265358979 0 3.14159265358979 -> xyz=0 -0.05085 -0.19574 rpy=3.14159265358979 0 3.14159265358979
- joint world_to_base_link: origin xyz=0 0 0 rpy=0 0 0 -> xyz=0 0 0 rpy=0 0 -1.57079632679
